Commit message: Final changes

File: src/urdf_files/my_robot.urdf (robot description, URDF)
Before this commit: robot my_robot, 3 links, 2 joints
Links:
- added link base_footprint
- added link castor_wheel_link; visual sphere radius=0.05
Joints:
- added joint base_castor_wheel_joint: type continuous, parent base_link, child castor_wheel_link, origin xyz=0.2 0 -0.05 rpy=0 0 0
- added joint base_joint: type fixed, parent base_footprint, child base_link, origin xyz=0 0 0.1 rpy=0 0 0
