Commit message: Adding Collision_tags

File: src/my_robot_description/urdf/mobile_base.xacro (robot description, xacro)
@@ -15,4 +15,10 @@
             <material name="violet"></material>
         </visual>
+        <collision>
+            <geometry>
+                <box size="${base_length} ${base_width} ${base_height}"></box>
+            </geometry>
+             <origin xyz="0 0 ${base_height / 2.0}" rpy="0 0 0"></origin>
+        </collision>
         <xacro:box_inertia m="5.0" x="${base_length}" y="${base_width}" z="${base_height}" o_xyz="0 0 ${base_height / 2.0}" o_rpy="0 0 0"></xacro:box_inertia>
     </link>
@@ -26,4 +32,10 @@
                 <material name="grey"></material>
             </visual>
+            <collision>
+                <geometry>
+                    <sphere radius="${wheel_radius}"></sphere>
+                </geometry>
+                <origin xyz="0 0 0" rpy="0 0 0"></origin>
+            </collision>
             <xacro:cylinder_inertia m="1.0" r="${wheel_radius}" l="${wheel_length}" o_xyz="0 0 0" o_rpy="${pi / 2.0} 0 0"></xacro:cylinder_inertia>
         </link>
@@ -39,4 +51,10 @@
             <material name="grey"></material>
         </visual>
+        <collision>
+            <geometry>
+                <sphere radius="${wheel_radius/2.0}"></sphere>
+            </geometry>
+            <origin xyz="0 0 0" rpy="0 0 0"></origin>
+        </collision>
         <xacro:sphere_inertia m="0.5" r="${wheel_radius/2.0}" o_xyz="0 0 0" o_rpy="0 0 0"></xacro:sphere_inertia>
     </link>

Commit message: Running robot

File: src/my_robot_description/urdf/mobile_base.xacro (robot description, xacro)
@@ -76,8 +76,8 @@
         <axis xyz="0 1 0"></axis>
     </joint>
-    <joint name="base_castor_wheel_joint" type="continuous">
-        <parent link="base_link"></parent>
-        <child link="castor_wheel_link"></child>
-        <origin xyz="${base_length / 3.00} 0 ${-(wheel_radius/2)}" rpy="0 0 0"></origin>
+    <joint name="base_castor_wheel_joint" type="fixed">
+        <parent link="base_link"/>
+        <child link="castor_wheel_link"/>
+        <origin xyz="${base_length / 3.00} 0 ${-(wheel_radius/2)}" rpy="0 0 0"/>
     </joint>
 </robot>

File: src/my_robot_description/urdf/mobile_base_gazebo.xacro (robot description, xacro)
@@ -9,6 +9,6 @@
         filename="gz-sim-diff-drive-system"
         name="gz::sim::systems::DiffDrive">
-            <left_join>base_left_wheel_joint</left_join>
-            <right_join>base_right_wheel_joint</right_join>
+            <left_joint>base_left_wheel_joint</left_joint>
+            <right_joint>base_right_wheel_joint</right_joint>
             <wheel_seperation>0.45</wheel_seperation>
             <wheel_radius>0.1</wheel_radius>

Commit message: Collision tag (#18)
* Adding Collision_tags

* Adding package for gazebo launch

* Adding gazebo config for URDF

* Running robot

File: src/my_robot_description/urdf/mobile_base.xacro (robot description, xacro)
@@ -15,4 +15,10 @@
             <material name="violet"></material>
         </visual>
+        <collision>
+            <geometry>
+                <box size="${base_length} ${base_width} ${base_height}"></box>
+            </geometry>
+             <origin xyz="0 0 ${base_height / 2.0}" rpy="0 0 0"></origin>
+        </collision>
         <xacro:box_inertia m="5.0" x="${base_length}" y="${base_width}" z="${base_height}" o_xyz="0 0 ${base_height / 2.0}" o_rpy="0 0 0"></xacro:box_inertia>
     </link>
@@ -26,4 +32,10 @@
                 <material name="grey"></material>
             </visual>
+            <collision>
+                <geometry>
+                    <sphere radius="${wheel_radius}"></sphere>
+                </geometry>
+                <origin xyz="0 0 0" rpy="0 0 0"></origin>
+            </collision>
             <xacro:cylinder_inertia m="1.0" r="${wheel_radius}" l="${wheel_length}" o_xyz="0 0 0" o_rpy="${pi / 2.0} 0 0"></xacro:cylinder_inertia>
         </link>
@@ -39,4 +51,10 @@
             <material name="grey"></material>
         </visual>
+        <collision>
+            <geometry>
+                <sphere radius="${wheel_radius/2.0}"></sphere>
+            </geometry>
+            <origin xyz="0 0 0" rpy="0 0 0"></origin>
+        </collision>
         <xacro:sphere_inertia m="0.5" r="${wheel_radius/2.0}" o_xyz="0 0 0" o_rpy="0 0 0"></xacro:sphere_inertia>
     </link>
@@ -58,8 +76,8 @@
         <axis xyz="0 1 0"></axis>
     </joint>
-    <joint name="base_castor_wheel_joint" type="continuous">
-        <parent link="base_link"></parent>
-        <child link="castor_wheel_link"></child>
-        <origin xyz="${base_length / 3.00} 0 ${-(wheel_radius/2)}" rpy="0 0 0"></origin>
+    <joint name="base_castor_wheel_joint" type="fixed">
+        <parent link="base_link"/>
+        <child link="castor_wheel_link"/>
+        <origin xyz="${base_length / 3.00} 0 ${-(wheel_radius/2)}" rpy="0 0 0"/>
     </joint>
 </robot>
