Commit message: Adding inertial prop

File: src/my_robot_description/urdf/common_properties.xacro (robot description, xacro)
@@ -7,3 +7,30 @@
         <color rgba="0.5 0.5 0.5 0.8"></color>
     </material>
+    <xacro:macro name="box_inertia" params="m x y z o_xyz o_rpy">
+        <inertial>
+            <mass value="${m}"></mass>
+            <origin xyz="${o_xyz}" rpy="${o_rpy}"></origin>
+            <inertia    ixx="${(m/12) *(y*y + z*z)}"    ixy="0" ixz="0"
+                        iyy="${(m/12) *(x*x + z*z)}"    iyz="0"
+                        izz="${(m/12) *(y*y + x*x)}"></inertia>
+        </inertial>
+    </xacro:macro>
+    <xacro:macro name="cylinder_inertia" params="m r l o_xyz o_rpy">
+        <inertial>
+            <mass value="${m}"></mass>
+            <origin xyz="${o_xyz}" rpy="${o_rpy}"></origin>
+            <inertia    ixx="${(m/12) *(3*r*r + l*l)}"    ixy="0" ixz="0"
+                        iyy="${(m/12) *(3*r*r + l*l)}"  iyz="0"
+                        izz="${(m/2) *(r*r)}"></inertia>
+        </inertial>
+    </xacro:macro>
+    <xacro:macro name="sphere_inertia" params="m r o_xyz o_rpy">
+        <inertial>
+            <mass value="${m}"></mass>
+            <origin xyz="${o_xyz}" rpy="${o_rpy}"></origin>
+            <inertia    ixx="${(2 * m/5) *(r*r)}"    ixy="0" ixz="0"
+                        iyy="${(2 * m/5) *(r*r)}"  iyz="0"
+                        izz="${(2 * m/5) *(r*r)}"></inertia>
+        </inertial>
+    </xacro:macro>
 </robot>

File: src/my_robot_description/urdf/mobile_base.xacro (robot description, xacro)
@@ -15,4 +15,5 @@
             <material name="violet"></material>
         </visual>
+        <xacro:box_inertia m="5.0" x="${base_length}" y="${base_width}" z="${base_height}" o_xyz="0 0 ${base_height / 2.0}" o_rpy="0 0 0"></xacro:box_inertia>
     </link>
     <xacro:macro name="wheel_link" params="prefix">
@@ -25,4 +26,5 @@
                 <material name="grey"></material>
             </visual>
+            <xacro:cylinder_inertia m="1.0" r="${wheel_radius}" l="${wheel_length}" o_xyz="0 0 0" o_rpy="${pi / 2.0} 0 0"></xacro:cylinder_inertia>
         </link>
     </xacro:macro>
@@ -37,4 +39,5 @@
             <material name="grey"></material>
         </visual>
+        <xacro:sphere_inertia m="0.5" r="${wheel_radius/2.0}" o_xyz="0 0 0" o_rpy="0 0 0"></xacro:sphere_inertia>
     </link>
     <joint name="base_joint" type="fixed">

Commit message: Adding URDF for robotic arm

File: src/my_robot_description/urdf/common_properties.xacro (robot description, xacro)
@@ -2,8 +2,14 @@
 <robot xmlns:xacro="https://www.ros.org/wiki/xacro">
     <material name="violet">
-        <color rgba="0.75 0.45 0.23 1"></color>
+        <color rgba="0.75 0.45 0.9 0.8"></color>
     </material>
     <material name="grey">
         <color rgba="0.5 0.5 0.5 0.8"></color>
+    </material>
+    <material name="orange">
+        <color rgba="1 0.5 0 0.8"></color>
+    </material>
+     <material name="yellow">
+        <color rgba="1 1 0 0.8"></color>
     </material>
     <xacro:macro name="box_inertia" params="m x y z o_xyz o_rpy">
