Commit message: Adding collision and Inertial tags

File: src/my_robot_description/urdf/arm.xacro (robot description, xacro)
@@ -16,4 +16,11 @@
             <material name="orange"></material>
         </visual>
+        <collision>
+            <geometry>
+                <box size="${arm_base_length} ${arm_base_width} ${arm_base_height}"></box>
+            </geometry>
+            <origin xyz="0 0 ${arm_base_height / 2.0}" rpy="0 0 0"></origin>
+        </collision>
+        <xacro:box_inertia m="0.5" x="${arm_base_length}" y="${arm_base_width}" z="${arm_base_height}" o_xyz="0 0 ${arm_base_height / 2.0}" o_rpy="0 0 0"></xacro:box_inertia>
     </link>
     <link name="forearm_link">
@@ -25,4 +32,11 @@
             <material name="yellow"></material>
         </visual>
+        <collision>
+            <geometry>
+                <cylinder radius="${forearm_radius}" length="${forearm_length}"></cylinder>
+            </geometry>
+            <origin xyz="0 0 ${forearm_length / 2.0}" rpy="0 0 0"></origin>
+        </collision>
+        <xacro:cylinder_inertia m="0.3" r="${forearm_radius}" l="${forearm_length}" o_xyz="0 0 ${forearm_length / 2.0}" o_rpy="0 0 0"></xacro:cylinder_inertia>
     </link>
     <link name="hand_link">
@@ -34,4 +48,11 @@
             <material name="orange"></material>
         </visual>
+        <collision>
+            <geometry>
+                <cylinder radius="${hand_radius}" length="${hand_length}"></cylinder>
+            </geometry>
+            <origin xyz="0 0 ${hand_length / 2.0}" rpy="0 0 0"></origin>
+        </collision>
+        <xacro:cylinder_inertia m="0.3" r="${hand_radius}" l="${hand_length}" o_xyz="0 0 ${hand_length / 2.0}" o_rpy="0 0 0"></xacro:cylinder_inertia>
     </link>
     <joint name="arm_base_forearm_joint" type="revolute">
@@ -41,4 +62,5 @@
         <axis xyz="0 1 0"></axis>
         <limit lower="0" upper="${pi / 2.0}" effort="100" velocity="100"></limit>
+        <dynamics friction="0.3" damping="0.3"></dynamics>
     </joint>
     <joint name="forearm_hand_joint" type="revolute">
@@ -48,4 +70,5 @@
         <axis xyz="0 1 0"></axis>
         <limit lower="0" upper="${pi / 2.0}" effort="100" velocity="100"></limit>
+        <dynamics friction="0.3" damping="0.3"></dynamics>
     </joint>
 </robot>
