Commit message: Adding xacro changes

File: src/my_robot_description/urdf/my_robot.urdf.xacro (robot description, xacro)
@@ -1,4 +1,4 @@
 <?xml version="1.0"?>
-<robot name="my_robot">
+<robot name="my_robot" xmlns:xacro="https://www.ros.org/wiki/xacro">
     <material name="violet">
         <color rgba="0.8 0.2 0.9 1"></color>
@@ -22,5 +22,5 @@
                 <cylinder radius="0.1" length="0.05"></cylinder>
             </geometry>
-            <origin xyz="0 0 0" rpy="1.57 0 0"></origin>
+            <origin xyz="0 0 0" rpy="${pi / 2.0} 0 0"></origin>
             <material name="grey"></material>
         </visual>

Commit message: Adding xacro constants

File: src/my_robot_description/urdf/my_robot.urdf.xacro (robot description, xacro)
@@ -1,6 +1,7 @@
 <?xml version="1.0"?>
 <robot name="my_robot" xmlns:xacro="https://www.ros.org/wiki/xacro">
+    <xacro:property name="base_length" value="0.60"></xacro:property>
     <material name="violet">
-        <color rgba="0.8 0.2 0.9 1"></color>
+        <color rgba="0.75 0.45 0.23 1"></color>
     </material>
     <material name="grey">
@@ -11,5 +12,5 @@
         <visual>
             <geometry>
-                <box size="0.6 0.4 0.2"></box>
+                <box size="${base_length} 0.4 0.2"></box>
             </geometry>
             <origin xyz="0 0 0.1" rpy="0 0 0"></origin>
@@ -31,5 +32,5 @@
                 <cylinder radius="0.1" length="0.05"></cylinder>
             </geometry>
-            <origin xyz="0 0 0" rpy="1.57 0 0"></origin>
+            <origin xyz="0 0 0" rpy="${pi / 2.0} 0 0"></origin>
             <material name="grey"></material>
         </visual>
@@ -52,5 +53,5 @@
         <parent link="base_link"></parent>
         <child link="right_wheel_link"></child>
-        <origin xyz="-0.15 -0.225 0" rpy="0 0 0"></origin>
+        <origin xyz="${-base_length / 4.00} -0.225 0" rpy="0 0 0"></origin>
         <axis xyz="0 1 0"></axis>
     </joint>
@@ -58,5 +59,5 @@
         <parent link="base_link"></parent>
         <child link="left_wheel_link"></child>
-        <origin xyz="-0.15 0.225 0" rpy="0 0 0"></origin>
+        <origin xyz="${-base_length / 4.00} 0.225 0" rpy="0 0 0"></origin>
         <axis xyz="0 1 0"></axis>
     </joint>
@@ -64,5 +65,5 @@
         <parent link="base_link"></parent>
         <child link="castor_wheel_link"></child>
-        <origin xyz="0.2 0 -0.05" rpy="0 0 0"></origin>
+        <origin xyz="${base_length / 3.00} 0 -0.05" rpy="0 0 0"></origin>
     </joint>
 </robot>

Commit message: Xacro adaptations (#14)
* Adding xacro changes

* Adding xacro constants

File: src/my_robot_description/urdf/my_robot.urdf.xacro (robot description, xacro)
@@ -1,6 +1,7 @@
 <?xml version="1.0"?>
-<robot name="my_robot">
+<robot name="my_robot" xmlns:xacro="https://www.ros.org/wiki/xacro">
+    <xacro:property name="base_length" value="0.60"></xacro:property>
     <material name="violet">
-        <color rgba="0.8 0.2 0.9 1"></color>
+        <color rgba="0.75 0.45 0.23 1"></color>
     </material>
     <material name="grey">
@@ -11,5 +12,5 @@
         <visual>
             <geometry>
-                <box size="0.6 0.4 0.2"></box>
+                <box size="${base_length} 0.4 0.2"></box>
             </geometry>
             <origin xyz="0 0 0.1" rpy="0 0 0"></origin>
@@ -22,5 +23,5 @@
                 <cylinder radius="0.1" length="0.05"></cylinder>
             </geometry>
-            <origin xyz="0 0 0" rpy="1.57 0 0"></origin>
+            <origin xyz="0 0 0" rpy="${pi / 2.0} 0 0"></origin>
             <material name="grey"></material>
         </visual>
@@ -31,5 +32,5 @@
                 <cylinder radius="0.1" length="0.05"></cylinder>
             </geometry>
-            <origin xyz="0 0 0" rpy="1.57 0 0"></origin>
+            <origin xyz="0 0 0" rpy="${pi / 2.0} 0 0"></origin>
             <material name="grey"></material>
         </visual>
@@ -52,5 +53,5 @@
         <parent link="base_link"></parent>
         <child link="right_wheel_link"></child>
-        <origin xyz="-0.15 -0.225 0" rpy="0 0 0"></origin>
+        <origin xyz="${-base_length / 4.00} -0.225 0" rpy="0 0 0"></origin>
         <axis xyz="0 1 0"></axis>
     </joint>
@@ -58,5 +59,5 @@
         <parent link="base_link"></parent>
         <child link="left_wheel_link"></child>
-        <origin xyz="-0.15 0.225 0" rpy="0 0 0"></origin>
+        <origin xyz="${-base_length / 4.00} 0.225 0" rpy="0 0 0"></origin>
         <axis xyz="0 1 0"></axis>
     </joint>
@@ -64,5 +65,5 @@
         <parent link="base_link"></parent>
         <child link="castor_wheel_link"></child>
-        <origin xyz="0.2 0 -0.05" rpy="0 0 0"></origin>
+        <origin xyz="${base_length / 3.00} 0 -0.05" rpy="0 0 0"></origin>
     </joint>
 </robot>

Commit message: Adding var for base

File: src/my_robot_description/urdf/my_robot.urdf.xacro (robot description, xacro)
@@ -2,4 +2,6 @@
 <robot name="my_robot" xmlns:xacro="https://www.ros.org/wiki/xacro">
     <xacro:property name="base_length" value="0.60"></xacro:property>
+    <xacro:property name="base_width" value="0.4"></xacro:property>
+    <xacro:property name="base_height" value="0.2"></xacro:property>
     <material name="violet">
         <color rgba="0.75 0.45 0.23 1"></color>
@@ -12,7 +14,7 @@
         <visual>
             <geometry>
-                <box size="${base_length} 0.4 0.2"></box>
+                <box size="${base_length} ${base_width} ${base_height}"></box>
             </geometry>
-            <origin xyz="0 0 0.1" rpy="0 0 0"></origin>
+            <origin xyz="0 0 ${base_height / 2.0}" rpy="0 0 0"></origin>
             <material name="violet"></material>
         </visual>
@@ -53,5 +55,5 @@
         <parent link="base_link"></parent>
         <child link="right_wheel_link"></child>
-        <origin xyz="${-base_length / 4.00} -0.225 0" rpy="0 0 0"></origin>
+        <origin xyz="${-base_length / 4.00} ${-(base_width+0.05)} 0" rpy="0 0 0"></origin>
         <axis xyz="0 1 0"></axis>
     </joint>
@@ -59,5 +61,5 @@
         <parent link="base_link"></parent>
         <child link="left_wheel_link"></child>
-        <origin xyz="${-base_length / 4.00} 0.225 0" rpy="0 0 0"></origin>
+        <origin xyz="${-base_length / 4.00} ${(base_width+0.05)} 0" rpy="0 0 0"></origin>
         <axis xyz="0 1 0"></axis>
     </joint>

Commit message: Adding vars

File: src/my_robot_description/urdf/my_robot.urdf.xacro (robot description, xacro)
@@ -1,7 +1,9 @@
 <?xml version="1.0"?>
 <robot name="my_robot" xmlns:xacro="https://www.ros.org/wiki/xacro">
-    <xacro:property name="base_length" value="0.60"></xacro:property>
+    <xacro:property name="base_length" value="0.6"></xacro:property>
     <xacro:property name="base_width" value="0.4"></xacro:property>
     <xacro:property name="base_height" value="0.2"></xacro:property>
+    <xacro:property name="wheel_radius" value="0.1"></xacro:property>
+    <xacro:property name="wheel_length" value="0.05"></xacro:property>
     <material name="violet">
         <color rgba="0.75 0.45 0.23 1"></color>
@@ -23,5 +25,5 @@
         <visual>
             <geometry>
-                <cylinder radius="0.1" length="0.05"></cylinder>
+                <cylinder radius="${wheel_radius}" length="${wheel_length}"></cylinder>
             </geometry>
             <origin xyz="0 0 0" rpy="${pi / 2.0} 0 0"></origin>
@@ -32,5 +34,5 @@
         <visual>
             <geometry>
-                <cylinder radius="0.1" length="0.05"></cylinder>
+                <cylinder radius="${wheel_radius}" length="${wheel_length}"></cylinder>
             </geometry>
             <origin xyz="0 0 0" rpy="${pi / 2.0} 0 0"></origin>
@@ -41,5 +43,5 @@
         <visual>
             <geometry>
-                <sphere radius="0.05"></sphere>
+                <sphere radius="${wheel_radius/2.0}"></sphere>
             </geometry>
             <origin xyz="0 0 0" rpy="0 0 0"></origin>
@@ -50,10 +52,10 @@
         <parent link="base_footprint"></parent>
         <child link="base_link"></child>
-        <origin xyz="0 0 0.1" rpy="0 0 0"></origin>
+        <origin xyz="0 0 ${wheel_radius}" rpy="0 0 0"></origin>
     </joint>
     <joint name="base_right_wheel_joint" type="continuous">
         <parent link="base_link"></parent>
         <child link="right_wheel_link"></child>
-        <origin xyz="${-base_length / 4.00} ${-(base_width+0.05)} 0" rpy="0 0 0"></origin>
+        <origin xyz="${-base_length / 4.00} ${-(base_width / 2+ wheel_length)} 0" rpy="0 0 0"></origin>
         <axis xyz="0 1 0"></axis>
     </joint>
@@ -61,5 +63,5 @@
         <parent link="base_link"></parent>
         <child link="left_wheel_link"></child>
-        <origin xyz="${-base_length / 4.00} ${(base_width+0.05)} 0" rpy="0 0 0"></origin>
+        <origin xyz="${-base_length / 4.00} ${(base_width / 2 + wheel_length)} 0" rpy="0 0 0"></origin>
         <axis xyz="0 1 0"></axis>
     </joint>
@@ -67,5 +69,5 @@
         <parent link="base_link"></parent>
         <child link="castor_wheel_link"></child>
-        <origin xyz="${base_length / 3.00} 0 -0.05" rpy="0 0 0"></origin>
+        <origin xyz="${base_length / 3.00} 0 ${-(wheel_radius/2)}" rpy="0 0 0"></origin>
     </joint>
 </robot>

Commit message: File level macros and includes

File: src/my_robot_description/urdf/my_robot.urdf.xacro (robot description, xacro)
@@ -1,73 +1,5 @@
 <?xml version="1.0"?>
 <robot name="my_robot" xmlns:xacro="https://www.ros.org/wiki/xacro">
-    <xacro:property name="base_length" value="0.6"></xacro:property>
-    <xacro:property name="base_width" value="0.4"></xacro:property>
-    <xacro:property name="base_height" value="0.2"></xacro:property>
-    <xacro:property name="wheel_radius" value="0.1"></xacro:property>
-    <xacro:property name="wheel_length" value="0.05"></xacro:property>
-    <material name="violet">
-        <color rgba="0.75 0.45 0.23 1"></color>
-    </material>
-    <material name="grey">
-        <color rgba="0.5 0.5 0.5 0.8"></color>
-    </material>
-    <link name="base_footprint"></link>
-    <link name="base_link">
-        <visual>
-            <geometry>
-                <box size="${base_length} ${base_width} ${base_height}"></box>
-            </geometry>
-            <origin xyz="0 0 ${base_height / 2.0}" rpy="0 0 0"></origin>
-            <material name="violet"></material>
-        </visual>
-    </link>
-    <link name="right_wheel_link">
-        <visual>
-            <geometry>
-                <cylinder radius="${wheel_radius}" length="${wheel_length}"></cylinder>
-            </geometry>
-            <origin xyz="0 0 0" rpy="${pi / 2.0} 0 0"></origin>
-            <material name="grey"></material>
-        </visual>
-    </link>
-    <link name="left_wheel_link">
-        <visual>
-            <geometry>
-                <cylinder radius="${wheel_radius}" length="${wheel_length}"></cylinder>
-            </geometry>
-            <origin xyz="0 0 0" rpy="${pi / 2.0} 0 0"></origin>
-            <material name="grey"></material>
-        </visual>
-    </link>
-    <link name="castor_wheel_link">
-        <visual>
-            <geometry>
-                <sphere radius="${wheel_radius/2.0}"></sphere>
-            </geometry>
-            <origin xyz="0 0 0" rpy="0 0 0"></origin>
-            <material name="grey"></material>
-        </visual>
-    </link>
-    <joint name="base_joint" type="fixed">
-        <parent link="base_footprint"></parent>
-        <child link="base_link"></child>
-        <origin xyz="0 0 ${wheel_radius}" rpy="0 0 0"></origin>
-    </joint>
-    <joint name="base_right_wheel_joint" type="continuous">
-        <parent link="base_link"></parent>
-        <child link="right_wheel_link"></child>
-        <origin xyz="${-base_length / 4.00} ${-(base_width / 2+ wheel_length)} 0" rpy="0 0 0"></origin>
-        <axis xyz="0 1 0"></axis>
-    </joint>
-    <joint name="base_left_wheel_joint" type="continuous">
-        <parent link="base_link"></parent>
-        <child link="left_wheel_link"></child>
-        <origin xyz="${-base_length / 4.00} ${(base_width / 2 + wheel_length)} 0" rpy="0 0 0"></origin>
-        <axis xyz="0 1 0"></axis>
-    </joint>
-    <joint name="base_castor_wheel_joint" type="continuous">
-        <parent link="base_link"></parent>
-        <child link="castor_wheel_link"></child>
-        <origin xyz="${base_length / 3.00} 0 ${-(wheel_radius/2)}" rpy="0 0 0"></origin>
-    </joint>
+    <xacro:include  filename="common_properties.xacro"></xacro:include>
+    <xacro:include  filename="mobile_base.xacro"></xacro:include>
 </robot>

Commit message: Xacro activity (#15)
* Adding var for base

* Adding vars

* File level macros and includes

File: src/my_robot_description/urdf/my_robot.urdf.xacro (robot description, xacro)
@@ -1,69 +1,5 @@
 <?xml version="1.0"?>
 <robot name="my_robot" xmlns:xacro="https://www.ros.org/wiki/xacro">
-    <xacro:property name="base_length" value="0.60"></xacro:property>
-    <material name="violet">
-        <color rgba="0.75 0.45 0.23 1"></color>
-    </material>
-    <material name="grey">
-        <color rgba="0.5 0.5 0.5 0.8"></color>
-    </material>
-    <link name="base_footprint"></link>
-    <link name="base_link">
-        <visual>
-            <geometry>
-                <box size="${base_length} 0.4 0.2"></box>
-            </geometry>
-            <origin xyz="0 0 0.1" rpy="0 0 0"></origin>
-            <material name="violet"></material>
-        </visual>
-    </link>
-    <link name="right_wheel_link">
-        <visual>
-            <geometry>
-                <cylinder radius="0.1" length="0.05"></cylinder>
-            </geometry>
-            <origin xyz="0 0 0" rpy="${pi / 2.0} 0 0"></origin>
-            <material name="grey"></material>
-        </visual>
-    </link>
-    <link name="left_wheel_link">
-        <visual>
-            <geometry>
-                <cylinder radius="0.1" length="0.05"></cylinder>
-            </geometry>
-            <origin xyz="0 0 0" rpy="${pi / 2.0} 0 0"></origin>
-            <material name="grey"></material>
-        </visual>
-    </link>
-    <link name="castor_wheel_link">
-        <visual>
-            <geometry>
-                <sphere radius="0.05"></sphere>
-            </geometry>
-            <origin xyz="0 0 0" rpy="0 0 0"></origin>
-            <material name="grey"></material>
-        </visual>
-    </link>
-    <joint name="base_joint" type="fixed">
-        <parent link="base_footprint"></parent>
-        <child link="base_link"></child>
-        <origin xyz="0 0 0.1" rpy="0 0 0"></origin>
-    </joint>
-    <joint name="base_right_wheel_joint" type="continuous">
-        <parent link="base_link"></parent>
-        <child link="right_wheel_link"></child>
-        <origin xyz="${-base_length / 4.00} -0.225 0" rpy="0 0 0"></origin>
-        <axis xyz="0 1 0"></axis>
-    </joint>
-    <joint name="base_left_wheel_joint" type="continuous">
-        <parent link="base_link"></parent>
-        <child link="left_wheel_link"></child>
-        <origin xyz="${-base_length / 4.00} 0.225 0" rpy="0 0 0"></origin>
-        <axis xyz="0 1 0"></axis>
-    </joint>
-    <joint name="base_castor_wheel_joint" type="continuous">
-        <parent link="base_link"></parent>
-        <child link="castor_wheel_link"></child>
-        <origin xyz="${base_length / 3.00} 0 -0.05" rpy="0 0 0"></origin>
-    </joint>
+    <xacro:include  filename="common_properties.xacro"></xacro:include>
+    <xacro:include  filename="mobile_base.xacro"></xacro:include>
 </robot>

Commit message: Stacking arm on top of robot

File: src/my_robot_description/urdf/my_robot.urdf.xacro (robot description, xacro)
@@ -5,3 +5,10 @@
     <xacro:include  filename="mobile_base_gazebo.xacro"></xacro:include>
     <xacro:include  filename="camera.xacro"></xacro:include>
+    <xacro:include  filename="arm.xacro"></xacro:include>
+    <xacro:include  filename="arm_gazebo.xacro"></xacro:include>
+    <joint name="mobile_base_arm_joint" type="fixed">
+        <parent link="base_link"></parent>
+        <child link="arm_base_link"></child>
+        <origin xyz="${base_length / 4.0} 0 ${base_height}" rpy="0 0 0"></origin>
+    </joint>
 </robot>
