Commit message: adding shoulder and joint

File: src/arm_robot/urdf/arm.urdf (robot description, URDF)
Before this commit: robot my_robot, 1 links, 0 joints
Links:
- added link shoulder_link; visual cylinder length=0.5 radius=0.1
Joints:
- added joint joint1: type revolute, parent base_link, child shoulder_link, origin xyz=0 0 0 rpy=0 0 0, axis 1 0 0, limit lower=-3.14 upper=3.14 effort=1000.0 velocity=1.0

Commit message: fixing origin of shoulder

File: src/arm_robot/urdf/arm.urdf (robot description, URDF)
Before this commit: robot my_robot, 2 links, 1 joints
Joints:
- joint joint1: origin xyz=0 0 0 rpy=0 0 0 -> xyz=0 0 0.1 rpy=0 0 0

Commit message: fixing rotation

File: src/arm_robot/urdf/arm.urdf (robot description, URDF)
Before this commit: robot my_robot, 2 links, 1 joints
Joints:
- joint joint1: axis 1 0 0 -> 0 0 1

Commit message: Adding all links and joints

File: src/arm_robot/urdf/arm.urdf (robot description, URDF)
Before this commit: robot my_robot, 2 links, 1 joints
Links:
- added link arm_link; visual cylinder length=0.6 radius=0.05
- added link elbow_link; visual cylinder length=0.1 radius=0.05
- added link forearm_link; visual cylinder length=0.5 radius=0.05
- added link hand_link; visual box size=0.1 0.1 0.02
- added link tool_link
- added link wrist_link; visual box size=0.1 0.1 0.05
Joints:
- added joint hand_tool_joint: type fixed, parent hand_link, child tool_link, origin xyz=0 0 0.02 rpy=0 0 0
- added joint joint2: type revolute, parent shoulder_link, child arm_link, origin xyz=0 0 0.5 rpy=0 0 0, axis 0 1 0, limit lower=0 upper=2.5 effort=1000.0 velocity=1.0
- added joint joint3: type revolute, parent arm_link, child elbow_link, origin xyz=0 0 0.6 rpy=0 0 0, axis 0 1 0, limit lower=0 upper=2.5 effort=1000.0 velocity=1.0
- added joint joint4: type revolute, parent elbow_link, child forearm_link, origin xyz=0 0 0.1 rpy=0 0 0, axis 0 0 1, limit lower=-3.14 upper=3.14 effort=1000.0 velocity=1.0
- added joint joint5: type revolute, parent forearm_link, child wrist_link, origin xyz=0 0 0.5 rpy=0 0 0, axis 0 1 0, limit lower=-1.57 upper=1.57 effort=1000.0 velocity=1.0
- added joint joint6: type continuous, parent wrist_link, child hand_link, origin xyz=0 0 0.05 rpy=0 0 0, axis 0 0 1
