Commit message: Migrating to Xacro

File: src/arm_robot/urdf/arm.xacro (robot description, xacro)
@@ -1,10 +1,4 @@
 <?xml version="1.0"?>
-<robot name="my_robot">
-    <material name="grey">
-        <color rgba="0.5 0.5 0.5 1"></color>
-    </material>
-    <material name="blue">
-        <color rgba="0 0 0.5 1"></color>
-    </material>
+<robot xmlns:xacro="http://www.ros.org/wiki/xacro">
     <link name = "base_link">
         <visual>
